File: wireMap/wireMap.kicad_pcb (KiCad board)
At the start: 2 copper layers, 68.6 x 53.3 mm, 8 parts, among them J1 Power, J2 Digital/PWM, J3 Analog, J4 Digital/PWM

Commit message: Upgrade PCB to KiCad v10 and update footprints
Bump wireMap.kicad_pcb to KiCad 10 (version/date and generator_version) and migrate PCB file formats (tenting/covering/plugging/capping/filling, normalized numeric formatting, simplified layer lists and named nets). Switch 3D models to KICAD10_3DMODEL_DIR (.step), update sheetfile to wireMap.kicad_sch and add unit/pin metadata. Replace Arduino mounting-hole footprints with Button_Switch_THT:SW_PUSH_6mm variants and update many footprint/pad definitions. Adjust project settings in wireMap.kicad_pro (zones, checks and defaults) and expand net inspector state in wireMap.kicad_prl. Adds local .lck lockfiles.
Parts:
- added REF**: SW_PUSH_6mm, Button_Switch_THT:SW_PUSH_6mm, F.Cu at (222.2, 93.8)
- added REF**: SW_PUSH_6mm, Button_Switch_THT:SW_PUSH_6mm, F.Cu at (256.8, 93.2)
- added REF**: SW_PUSH_6mm, Button_Switch_THT:SW_PUSH_6mm, F.Cu at (222.2, 54.8)
- added REF**: SW_PUSH_6mm, Button_Switch_THT:SW_PUSH_6mm, F.Cu at (204.5, 94.0)
- added REF**: SW_PUSH_6mm, Button_Switch_THT:SW_PUSH_6mm, F.Cu at (204.5, 81.5)
- added REF**: SW_PUSH_6mm, Button_Switch_THT:SW_PUSH_6mm, F.Cu at (239.0, 67.0)
- added REF**: SW_PUSH_6mm, Button_Switch_THT:SW_PUSH_6mm, F.Cu at (239.0, 93.5)
- added REF**: SW_PUSH_6mm, Button_Switch_THT:SW_PUSH_6mm, F.Cu at (204.5, 55.0)
- added REF**: SW_PUSH_6mm, Button_Switch_THT:SW_PUSH_6mm, F.Cu at (256.8, 54.2)
- added REF**: SW_PUSH_6mm, Button_Switch_THT:SW_PUSH_6mm, F.Cu at (239.0, 81.0)
- added REF**: SW_PUSH_6mm, Button_Switch_THT:SW_PUSH_6mm, F.Cu at (222.2, 81.2)
- added REF**: SW_PUSH_6mm, Button_Switch_THT:SW_PUSH_6mm, F.Cu at (239.0, 54.5)
- added REF**: SW_PUSH_6mm, Button_Switch_THT:SW_PUSH_6mm, F.Cu at (256.8, 80.8)
- added REF**: SW_PUSH_6mm, Button_Switch_THT:SW_PUSH_6mm, F.Cu at (222.2, 67.2)
- added REF**: SW_PUSH_6mm, Button_Switch_THT:SW_PUSH_6mm, F.Cu at (256.8, 66.8)
- added REF**: SW_PUSH_6mm, Button_Switch_THT:SW_PUSH_6mm, F.Cu at (204.5, 67.5)
