File: hardware/wiring/wireMap/wireMap.kicad_sch (KiCad schematic)
At the start: 20 parts, among them J1 Power, J2 Digital/PWM, J3 Analog, J4 Digital/PWM, SW1 SW_Push, SW10 SW_Push, SW11 SW_Push, SW12 SW_Push, SW13 SW_Push, SW14 SW_Push, SW15 SW_Push, SW16 SW_Push, SW2 SW_Push, SW3 SW_Push, SW4 SW_Push, SW5 SW_Push, SW6 SW_Push, SW7 SW_Push, SW8 SW_Push, SW9 SW_Push

Commit message: Added diodes and updated wire plan SVG
Added diodes and updated wire plan SVG
Parts:
- added D1, D10, D11, D12, D13, D14, D15, D16, D2, D3, D4, D5, D6, D7, D8, D9: 1N4148, Diode_THT:D_DO-35_SOD27_P7.62mm_Horizontal, symbol Diode:1N4148
Connections:
- net *3: now also D10.1 (K), D11.1 (K), D12.1 (K), D9.1 (K); no longer SW10.2, SW15.2, SW5.2, SW6.2
- net *5: now also D1.1 (K), D2.1 (K), D3.1 (K), D4.1 (K); no longer SW1.2, SW12.2, SW13.2, SW2.2
- net 2: now also D13.1 (K), D14.1 (K), D15.1 (K), D16.1 (K); no longer SW11.2, SW16.2, SW7.2, SW8.2
- net 4: now also D5.1 (K), D6.1 (K), D7.1 (K), D8.1 (K); no longer SW14.2, SW3.2, SW4.2, SW9.2
- new net: D2.2 (A), SW2.2
- new net: D5.2 (A), SW3.2
- new net: D4.2 (A), SW13.2
- new net: D12.2 (A), SW15.2
- new net: D8.2 (A), SW14.2
- new net: D7.2 (A), SW9.2
- new net: D16.2 (A), SW16.2
- new net: D10.2 (A), SW6.2
- new net: D6.2 (A), SW4.2
- new net: D11.2 (A), SW10.2
- new net: D15.2 (A), SW11.2
- new net: D1.2 (A), SW1.2
- new net: D13.2 (A), SW7.2
- new net: D9.2 (A), SW5.2
- new net: D3.2 (A), SW12.2
- new net: D14.2 (A), SW8.2
